File: pcb/kicadproject.kicad_pcb (KiCad board)
At the start: 2 copper layers, 79.9 x 62 mm, 12 parts, among them SW1 SW_Push, SW2 SW_Push, SW3 SW_Push, SW4 SW_Push, SW5 SW_Push, SW6 SW_Push, SW7 RotaryEncoder_Switch, U1 XIAO-RP2040-DIP, U2 OLED_0.91_128x32

Commit message: updated
Connections:
- SW7 pad A: Net-(U1-3V3) -> Net-(U1-GPIO3/MOSI)
- SW7 pad B: Net-(U1-GPIO3/MOSI) -> Net-(U1-GPIO4/MISO)
- SW7 pad S1: Net-(U1-GPIO4/MISO) -> unconnected-(SW7-PadS1)
- U1 pad 12: Net-(U1-3V3) -> unconnected-(U1-3V3-Pad12)
Routing:
- net Net-(U1-3V3): track 143.3 -> 0.00 mm
- net Net-(U1-GPIO4/MISO): track 67.0 -> 52.5 mm
- net Net-(U1-GPIO3/MOSI): track 55.0 -> 58.5 mm, vias 0 -> 1
Changed lines of the file:
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@@
 			(outputformat 1)
 			(mirror no)
-			(drillshape 1)
+			(drillshape 0)
 			(scaleselection 1)
-			(outputdirectory "")
+			(outputdirectory "../../../cherrystreampad/production/gerber/")
 		)
 	)
@@
 	(net 12 "Net-(U1-GPIO6{slash}SDA)")
 	(net 13 "Net-(U1-GPIO29{slash}ADC3{slash}A3)")
-	(net 14 "Net-(U1-3V3)")
+	(net 14 "unconnected-(SW7-PadS1)")
 	(net 15 "Net-(U1-GPIO28{slash}ADC2{slash}A2)")
 	(net 16 "Net-(U1-GPIO27{slash}ADC1{slash}A1)")
+	(net 17 "unconnected-(U1-3V3-Pad12)")
 	(footprint "LED_SMD:LED_SK6812MINI_PLCC4_3.5x3.5mm_P1.75mm"
 		(layer "F.Cu")
@@
 			(layers "*.Cu" "*.Mask")
 			(remove_unused_layers no)
-			(net 14 "Net-(U1-3V3)")
+			(net 9 "Net-(U1-GPIO3{slash}MOSI)")
 			(pinfunction "A")
 			(pintype "passive")
@@
 			(layers "*.Cu" "*.Mask")
 			(remove_unused_layers no)
-			(net 9 "Net-(U1-GPIO3{slash}MOSI)")
+			(net 8 "Net-(U1-GPIO4{slash}MISO)")
 			(pinfunction "B")
 			(pintype "passive")
@@
 			(layers "*.Cu" "*.Mask")
 			(remove_unused_layers no)
-			(net 8 "Net-(U1-GPIO4{slash}MISO)")
+			(net 14 "unconnected-(SW7-PadS1)")
 			(pinfunction "S1")
 			(pintype "passive")
@@
 			)
 		)
-		(property "Description" "XIAO HERE!"
+		(property "Description" ""
 			(at 0 0 90)
 			(unlocked yes)
@@
 			(layers "*.Cu" "*.Mask")
 			(remove_unused_layers no)
-			(net 14 "Net-(U1-3V3)")
+			(net 17 "unconnected-(U1-3V3-Pad12)")
 			(pinfunction "3V3")
 			(pintype "passive")
@@
 			(layers "B.Cu" "B.Mask")
 			(roundrect_rratio 0.1)
-			(net 14 "Net-(U1-3V3)")
+			(net 17 "unconnected-(U1-3V3-Pad12)")
 			(pinfunction "3V3")
 			(pintype "passive")
@@
 	)
 	(segment
-		(start 88.70365 58.52075)
+		(start 127.29 61)
 		(end 91.1829 61)
 		(width 0.2)
@@
 	)
 	(segment
-		(start 141.79 61)
-		(end 146.315 56.475)
+		(start 88.70365 58.52075)
+		(end 91.1829 61)
 		(width 0.2)
 		(layer "F.Cu")
@@
 	)
 	(segment
-		(start 91.1829 61)
-		(end 141.79 61)
+		(start 131.815 56.475)
+		(end 127.29 61)
 		(width 0.2)
 		(layer "F.Cu")
@@
 	)
 	(segment
-		(start 82.14075 58.11975)
-		(end 88.86975 58.11975)
+		(start 125.9 59.9)
+		(end 125.6 60.2)
 		(width 0.2)
 		(layer "F.Cu")
@@
 	)
 	(segment
-		(start 91.25 60.5)
-		(end 127.79 60.5)
+		(start 82.1605 58.1)
+		(end 80.27575 59.98475)
 		(width 0.2)
 		(layer "F.Cu")
@@
 	)
 	(segment
-		(start 127.79 60.5)
-		(end 131.815 56.475)
+		(start 90.639196 58.1)
+		(end 82.1605 58.1)
 		(width 0.2)
 		(layer "F.Cu")
@@
 	)
 	(segment
-		(start 80.27575 59.98475)
-		(end 82.14075 58.11975)
+		(start 92.739196 60.2)
+		(end 90.639196 58.1)
 		(width 0.2)
 		(layer "F.Cu")
@@
 	)
 	(segment
-		(start 88.86975 58.11975)
-		(end 91.25 60.5)
+		(start 125.6 60.2)
+		(end 92.739196 60.2)
 		(width 0.2)
 		(layer "F.Cu")
 		(net 9)
 	)
+	(via
+		(at 125.9 59.9)
+		(size 0.6)
+		(drill 0.3)
+		(layers "F.Cu" "B.Cu")
+		(net 9)
+	)
+	(segment
+		(start 125.9 57.39)
+		(end 125.9 59.9)
+		(width 0.2)
+		(layer "B.Cu")
+		(net 9)
+	)
+	(segment
+		(start 131.815 51.475)
+		(end 125.9 57.39)
+		(width 0.2)
+		(layer "B.Cu")
+		(net 9)
+	)
+	(segment
+		(start 125.9 59.9)
+		(end 125.9 60.1)
+		(width 0.2)
+		(layer "B.Cu")
+		(net 9)
+	)
 	(segment
 		(start 87.89575 44.74475)
@@
 	)
 	(segment
-		(start 89.726184 94.351)
-		(end 77.73575 82.360566)
-		(width 0.2)
-		(layer "F.Cu")
-		(net 14)
-	)
-	(segment
-		(start 77.73575 82.360566)
-		(end 77.73575 59.98475)
-		(width 0.2)
-		(layer "F.Cu")
-		(net 14)
-	)
-	(segment
-		(start 148.017 51.337108)
-		(end 148.017 67.213686)
-		(width 0.2)
-		(layer "F.Cu")
-		(net 14)
-	)
-	(segment
-		(start 126.341 90.050314)
-		(end 125.520314 90.871)
-		(width 0.2)
-		(layer "F.Cu")
-		(net 14)
-	)
-	(segment
-		(start 126.341 88.889686)
-		(end 126.341 90.050314)
-		(width 0.2)
-		(layer "F.Cu")
-		(net 14)
-	)
-	(segment
-		(start 123.539 90.050314)
-		(end 119.238314 94.351)
-		(width 0.2)
-		(layer "F.Cu")
-		(net 14)
-	)
-	(segment
-		(start 124.359686 90.871)
-		(end 123.539 90.050314)
-		(width 0.2)
-		(layer "F.Cu")
-		(net 14)
-	)
-	(segment
-		(start 131.815 51.475)
-		(end 133.116 50.174)
-		(width 0.2)
-		(layer "F.Cu")
-		(net 14)
-	)
-	(segment
-		(start 146.853892 50.174)
-		(end 148.017 51.337108)
-		(width 0.2)
-		(layer "F.Cu")
-		(net 14)
-	)
-	(segment
-		(start 125.520314 90.871)
-		(end 124.359686 90.871)
-		(width 0.2)
-		(layer "F.Cu")
-		(net 14)
-	)
-	(segment
-		(start 148.017 67.213686)
-		(end 126.341 88.889686)
-		(width 0.2)
-		(layer "F.Cu")
-		(net 14)
-	)
-	(segment
-		(start 133.116 50.174)
-		(end 146.853892 50.174)
-		(width 0.2)
-		(layer "F.Cu")
-		(net 14)
-	)
-	(segment
-		(start 119.238314 94.351)
-		(end 89.726184 94.351)
-		(width 0.2)
-		(layer "F.Cu")
-		(net 14)
-	)
-	(segment
