File: pcb/kicadproject.kicad_sch (KiCad schematic)
At the start: 11 parts, among them SW1 SW_Push, SW2 SW_Push, SW3 SW_Push, SW4 SW_Push, SW5 SW_Push, SW6 SW_Push, SW7 RotaryEncoder_Switch, U1 XIAO-RP2040-DIP, U2 OLED_0.91_128x32

Commit message: updated
Connections:
- net at U1.10 (GPIO4/MISO): now also SW7.B; no longer SW7.S1
- net at U1.11 (GPIO3/MOSI): now also SW7.A; no longer SW7.B
- net at U1.12 (3V3): no longer SW7.A
Changed lines of the file:
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@@
-	(wire
-		(pts
-			(xy 223.52 82.55) (xy 223.52 115.57)
-		)
-		(stroke
-			(width 0)
-			(type default)
-		)
-	)
 	(wire
 		(pts
@@
 	(wire
 		(pts
+			(xy 193.04 87.63) (xy 193.04 115.57)
+		)
+		(stroke
+			(width 0)
+			(type default)
+		)
+	)
+	(wire
+		(pts
 			(xy 83.82 143.51) (xy 83.82 148.59)
 		)
@@
 	(wire
 		(pts
+			(xy 193.04 115.57) (xy 149.86 115.57)
+		)
+		(stroke
+			(width 0)
+			(type default)
+		)
+	)
+	(wire
+		(pts
 			(xy 116.84 81.28) (xy 149.86 81.28)
 		)
@@
 	(wire
 		(pts
-			(xy 208.28 82.55) (xy 223.52 82.55)
-		)
-		(stroke
-			(width 0)
-			(type default)
-		)
-	)
-	(wire
-		(pts
 			(xy 100.33 143.51) (xy 100.33 160.02)
 		)
@@
 	(wire
 		(pts
-			(xy 149.86 111.76) (xy 193.04 111.76)
-		)
-		(stroke
-			(width 0)
-			(type default)
-		)
-	)
-	(wire
-		(pts
 			(xy 193.04 82.55) (xy 177.8 82.55)
 		)
@@
 	(wire
 		(pts
+			(xy 149.86 111.76) (xy 177.8 111.76)
+		)
+		(stroke
+			(width 0)
+			(type default)
+		)
+	)
+	(wire
+		(pts
 			(xy 58.42 67.31) (xy 62.23 67.31)
 		)
@@
 	(wire
 		(pts
-			(xy 177.8 107.95) (xy 149.86 107.95)
-		)
-		(stroke
-			(width 0)
-			(type default)
-		)
-	)
-	(wire
-		(pts
 			(xy 156.21 119.38) (xy 149.86 119.38)
 		)
@@
 	(wire
 		(pts
+			(xy 177.8 111.76) (xy 177.8 82.55)
+		)
+		(stroke
+			(width 0)
+			(type default)
+		)
+	)
+	(wire
+		(pts
 			(xy 60.96 72.39) (xy 60.96 104.14)
 		)
@@
 	(wire
 		(pts
-			(xy 177.8 82.55) (xy 177.8 107.95)
-		)
-		(stroke
-			(width 0)
-			(type default)
-		)
-	)
-	(wire
-		(pts
 			(xy 107.95 73.66) (xy 109.22 73.66)
 		)
@@
 	(wire
 		(pts
-			(xy 193.04 111.76) (xy 193.04 87.63)
-		)
-		(stroke
-			(width 0)
-			(type default)
-		)
-	)
-	(wire
-		(pts
 			(xy 73.66 148.59) (xy 63.5 148.59)
 		)
@@
 		)
 		(stroke
-			(width 0)
-			(type default)
-		)
-	)
-	(wire
-		(pts
-			(xy 149.86 115.57) (xy 223.52 115.57)
-		)
-		(stroke
