File: pcb/kicadproject-2.kicad_pcb (KiCad board)
At the start: 2 copper layers, 79.9 x 62 mm, 12 parts, among them SW1 SW_Push, SW2 SW_Push, SW3 SW_Push, SW4 SW_Push, SW5 SW_Push, SW6 SW_Push, SW7 RotaryEncoder_Switch, U1 XIAO-RP2040-DIP, U2 OLED_0.91_128x32

Commit message: removedledaddedswitch
Parts:
- removed D1, D2: SK6812MINI, LED_SMD:LED_SK6812MINI_PLCC4_3.5x3.5mm_P1.75mm
Connections:
- SW7 pad S1: unconnected-(SW7-PadS1) -> Net-(U1-GPIO26/ADC0/A0)
- U1 pad 1: Net-(D1-DIN) -> Net-(U1-GPIO26/ADC0/A0)
Routing:
- net Net-(U1-GPIO26/ADC0/A0): track 0.00 -> 94.6 mm
- net Net-(D1-DIN): track 56.8 -> 0.00 mm
- net +5V: track 60.6 -> 26.6 mm
- net Net-(D1-DOUT): track 11.5 -> 0.00 mm
- net Net-(U1-GPIO7/SCL): track 53.4 -> 47.8 mm
- net Net-(U1-GPIO28/ADC2/A2): track 30.0 -> 27.6 mm
- net GND: track 209.2 -> 208.6 mm

Commit message: fixedpcb
Connections:
- SW4 pad 1: Net-(U1-GPIO7/SCL) -> Net-(U1-GPIO29/ADC3/A3)
- SW5 pad 1: Net-(U1-GPIO6/SDA) -> Net-(U1-GPIO28/ADC2/A2)
- SW6 pad 1: Net-(U1-GPIO29/ADC3/A3) -> Net-(U1-GPIO27/ADC1/A1)
- U2 pad 3: Net-(U1-GPIO28/ADC2/A2) -> Net-(U1-GPIO7/SCL)
- U2 pad 4: Net-(U1-GPIO27/ADC1/A1) -> Net-(U1-GPIO6/SDA)
Routing:
- net Net-(U1-GPIO27/ADC1/A1): track 38.0 -> 106.7 mm
- net GND: track 208.6 -> 153.8 mm
- net Net-(U1-GPIO6/SDA): track 63.2 -> 15.6 mm, vias 1 -> 0
- net Net-(U1-GPIO28/ADC2/A2): track 27.6 -> 69.2 mm
- net Net-(U1-GPIO7/SCL): track 47.8 -> 19.9 mm
- net Net-(U1-GPIO29/ADC3/A3): track 75.6 -> 53.0 mm, vias 1 -> 0
- net Net-(U1-GPIO2/SCK): track 25.8 -> 35.4 mm
- net +5V: track 26.6 -> 22.0 mm, vias 1 -> 0
- net Net-(U1-GPIO3/MOSI): track 58.3 -> 55.1 mm, vias 1 -> 0
- net Net-(U1-GPIO4/MISO): track 52.5 -> 50.5 mm
- net Net-(U1-GPIO0/TX): vias 1 -> 0
